Commit message: bracing for energy efficiency in contact and non contact tasks

File: 04-free_space_2d_bracing/4rbot_fixed.urdf (robot description, URDF)
Before this commit: robot 4pbot, 5 links, 4 joints
Links:
- link link0: geometry visual cylinder length=0.04 radius=0.1
- link link1: geometry visual box size=0.04 1.0 0.10; visual cylinder length=0.04 radius=0.1
- link link2: geometry collision cylinder length=0.04 radius=0.1; visual box size=0.04 1.0 0.10
- link link3: geometry visual box size=0.04 1.0 0.10; visual cylinder length=0.04 radius=0.1
- link link4: geometry visual box size=0.04 1.0 0.10; visual cylinder length=0.04 radius=0.1
Joints:
- joint j0: origin xyz=0.000000 0.000000 1.000000 rpy=-0.000000 0.000000 -0.000000 -> xyz=0.000000 0.000000 0.000000 rpy=-0.000000 0.000000 -0.000000
- joint j1: origin xyz=0.000000 0.000000 1.000000 rpy=-0.000000 0.000000 -0.000000 -> xyz=0.000000 1.000000 0.000000 rpy=-0.000000 0.000000 -0.000000
- joint j2: origin xyz=0.000000 0.000000 1.000000 rpy=-0.000000 0.000000 -0.000000 -> xyz=0.000000 1.000000 0.000000 rpy=-0.000000 0.000000 -0.000000
- joint j3: origin xyz=0.000000 0.000000 1.000000 rpy=-0.000000 0.000000 -0.000000 -> xyz=0.000000 1.000000 0.000000 rpy=-0.000000 0.000000 -0.000000

File: 05-contact_task_2d_bracing/4rbot_fixed.urdf (robot description, URDF)
Before this commit: robot 4pbot, 5 links, 4 joints
Links:
- link link0: geometry visual cylinder length=0.04 radius=0.1
- link link1: geometry visual box size=0.04 1.0 0.10; visual cylinder length=0.04 radius=0.1
- link link2: geometry collision cylinder length=0.04 radius=0.1; visual box size=0.04 1.0 0.10
- link link3: geometry visual box size=0.04 1.0 0.10; visual cylinder length=0.04 radius=0.1
- link link4: geometry collision cylinder length=0.04 radius=0.1; visual box size=0.04 1.0 0.10
Joints:
- joint j0: origin xyz=0.000000 0.000000 1.000000 rpy=-0.000000 0.000000 -0.000000 -> xyz=0.000000 0.000000 0.000000 rpy=-0.000000 0.000000 -0.000000
- joint j1: origin xyz=0.000000 0.000000 1.000000 rpy=-0.000000 0.000000 -0.000000 -> xyz=0.000000 1.000000 0.000000 rpy=-0.000000 0.000000 -0.000000
- joint j2: origin xyz=0.000000 0.000000 1.000000 rpy=-0.000000 0.000000 -0.000000 -> xyz=0.000000 1.000000 0.000000 rpy=-0.000000 0.000000 -0.000000
- joint j3: origin xyz=0.000000 0.000000 1.000000 rpy=-0.000000 0.000000 -0.000000 -> xyz=0.000000 1.000000 0.000000 rpy=-0.000000 0.000000 -0.000000
